Commit message: camera set, power set

File: urdf/ur5_robot.urdf.xacro (robot description, xacro)
@@ -15,69 +15,8 @@
   <xacro:golf_club prefix="" connected_to="tool0" />
   <!-- camera link -->
-  <link name="camera_link">
-    <visual>
-      <origin xyz="0 0 0" rpy="0 0 0"/>
-      <geometry>
-        <box size="0.1 0.1 0.1"/>
-      </geometry>
-      <material name="orange"/>
-    </visual>
-    <inertial>
-      <origin xyz="0 0 1" rpy="0 0 0"/>
-      <mass value="0.1"/>
-      <inertia
-        ixx="0.1" ixy="0.0" ixz="0.0"
-        iyy="0.1" iyz="0.0"
-        izz="0.1"/>
-    </inertial>
-  </link>
-  <gazebo reference="camera_link">
-    <sensor name="camera" type="depth">
-      <update_rate>20</update_rate>
-      <camera>
-        <horizontal_fov>1.047198</horizontal_fov>
-        <image>
-          <width>640</width>
-          <height>480</height>
-          <format>R8G8B8</format>
-        </image>
-        <clip>
-          <near>0.05</near>
-          <far>3</far>
-        </clip>
-      </camera>
-      <plugin name="camera_plugin" filename="libgazebo_ros_openni_kinect.so">
-        <baseline>0.2</baseline>
-        <alwaysOn>true</alwaysOn>
-        <!-- Keep this zero, update_rate in the parent <sensor> tag
-          will control the frame rate. -->
-        <updateRate>0.0</updateRate>
-        <cameraName>camera_ir</cameraName>
-        <imageTopicName>/camera/color/image_raw</imageTopicName>
-        <cameraInfoTopicName>/camera/color/camera_info</cameraInfoTopicName>
-        <depthImageTopicName>/camera/depth/image_raw</depthImageTopicName>
-        <depthImageCameraInfoTopicName>/camera/depth/camera_info</depthImageCameraInfoTopicName>
-        <pointCloudTopicName>/camera/depth/points</pointCloudTopicName>
-        <frameName>camera_link</frameName>
-        <pointCloudCutoff>0.5</pointCloudCutoff>
-        <pointCloudCutoffMax>3.0</pointCloudCutoffMax>
-        <distortionK1>0</distortionK1>
-        <distortionK2>0</distortionK2>
-        <distortionK3>0</distortionK3>
-        <distortionT1>0</distortionT1>
-        <distortionT2>0</distortionT2>
-        <CxPrime>0</CxPrime>
-        <Cx>0</Cx>
-        <Cy>0</Cy>
-        <focalLength>0</focalLength>
-        <hackBaseline>0</hackBaseline>
-      </plugin>
-    </sensor>
-  </gazebo>
-  <joint name="camera_joint" type="fixed">
-    <parent link="tool0" />
-    <child link = "camera_link" />
-    <origin xyz="0.0 0.0 0.0" rpy="0.0 ${-pi/2} ${pi/2}" />
-  </joint>
+  <xacro:include filename="$(find golfbot)/urdf/_d435.urdf.xacro" />
+  <xacro:sensor_d435 name="camera" topics_ns="camera" parent="world" publish_pointcloud="true">
+    <origin xyz="0 0 0.4" rpy="0 0 ${pi/2}" />
+  </xacro:sensor_d435>
   <link name="world" />
   <joint name="world_joint" type="fixed">
