Commit message: import meshes

File: urdf/golf_club.urdf.xacro (robot description, xacro)
@@ -11,8 +11,12 @@
                 <origin rpy="0 0 0" xyz="0 0 0" />
                 <geometry>
-                    <box size="0.05 0.05 0.05" />
+                    <mesh filename="package://golfbot/meshes/golf_club.stl"/>
                 </geometry>
-                <material name="green"/>
             </visual>
+            <collision>
+                <geometry>
+                    <mesh filename="package://golfbot/meshes/golf_club.stl"/>
+                </geometry>
+            </collision>
         </link>
     </xacro:macro>

Commit message: working the first time

File: urdf/golf_club.urdf.xacro (robot description, xacro)
@@ -9,12 +9,13 @@
         <link name="${prefix}_golf_club">
             <visual>
-                <origin rpy="0 0 0" xyz="0 0 0" />
+                <origin rpy="${pi/2} ${pi/2} 0" xyz="-0.1 0.5 0.1" />
                 <geometry>
-                    <mesh filename="package://golfbot/meshes/golf_club.stl"/>
+                    <mesh scale="0.005 0.005 0.005" filename="package://golfbot/meshes/golf_club.stl"/>
                 </geometry>
             </visual>
             <collision>
+                <origin rpy="${pi/2} ${pi/2} 0" xyz="-0.1 0.5 0.1" />
                 <geometry>
-                    <mesh filename="package://golfbot/meshes/golf_club.stl"/>
+                    <mesh scale="0.005 0.005 0.005" filename="package://golfbot/meshes/golf_club.stl"/>
                 </geometry>
             </collision>

Commit message: add swing and tee

File: urdf/golf_club.urdf.xacro (robot description, xacro)
@@ -9,5 +9,5 @@
         <link name="${prefix}_golf_club">
             <visual>
-                <origin rpy="${pi/2} ${pi/2} 0" xyz="-0.1 0.5 0.1" />
+                <origin rpy="${pi} ${pi/2} 0" xyz="0.0 0.6 0.0" />
                 <geometry>
                     <mesh scale="0.005 0.005 0.005" filename="package://golfbot/meshes/golf_club.stl"/>
@@ -15,5 +15,5 @@
             </visual>
             <collision>
-                <origin rpy="${pi/2} ${pi/2} 0" xyz="-0.1 0.5 0.1" />
+                <origin rpy="${pi} ${pi/2} 0" xyz="0.0 0.6 0.0" />
                 <geometry>
                     <mesh scale="0.005 0.005 0.005" filename="package://golfbot/meshes/golf_club.stl"/>

Commit message: working and added camera

File: urdf/golf_club.urdf.xacro (robot description, xacro)
@@ -19,5 +19,15 @@
                     <mesh scale="0.005 0.005 0.005" filename="package://golfbot/meshes/golf_club.stl"/>
                 </geometry>
+                <surface>
+                    <bounce>
+                        <restitution_coefficient>0.9</restitution_coefficient>
+                        <threshold>0</threshold>
+                    </bounce>
+                </surface>
             </collision>
+            <inertial>
+                <mass value="10"/>
+                <inertia ixx="10.0" ixy="0.0" ixz="0.0" iyy="0.0" iyz="0.0" izz="10.0"/>
+            </inertial>
         </link>
     <gazebo reference="${prefix}_golf_club">

File: urdf/ur5_robot.urdf.xacro (robot description, xacro)
@@ -6,5 +6,5 @@
   <xacro:include filename="$(find ur_description)/urdf/common.gazebo.xacro" />
   <!-- ur5 -->
-  <xacro:include filename="$(find ur_description)/urdf/ur5.urdf.xacro" />
+  <xacro:include filename="$(find golfbot)/urdf/ur5.urdf.xacro" />
   <xacro:include filename="golf_club.urdf.xacro" />
   <!-- arm -->
@@ -12,5 +12,72 @@
     transmission_hw_interface="$(arg transmission_hw_interface)"
   />
+  <!-- golf club -->
   <xacro:golf_club prefix="" connected_to="tool0" />
+  <!-- camera link -->
+  <link name="camera_link">
+    <visual>
+      <origin xyz="0 0 0" rpy="0 0 0"/>
+      <geometry>
+        <box size="0.1 0.1 0.1"/>
+      </geometry>
+      <material name="orange"/>
+    </visual>
+    <inertial>
+      <origin xyz="0 0 1" rpy="0 0 0"/>
+      <mass value="0.1"/>
+      <inertia
+        ixx="0.1" ixy="0.0" ixz="0.0"
+        iyy="0.1" iyz="0.0"
+        izz="0.1"/>
+    </inertial>
+  </link>
+  <gazebo reference="camera_link">
+    <sensor name="camera" type="depth">
+      <update_rate>20</update_rate>
+      <camera>
+        <horizontal_fov>1.047198</horizontal_fov>
+        <image>
+          <width>640</width>
+          <height>480</height>
+          <format>R8G8B8</format>
+        </image>
+        <clip>
+          <near>0.05</near>
+          <far>3</far>
+        </clip>
+      </camera>
+      <plugin name="camera_plugin" filename="libgazebo_ros_openni_kinect.so">
+        <baseline>0.2</baseline>
+        <alwaysOn>true</alwaysOn>
+        <!-- Keep this zero, update_rate in the parent <sensor> tag
+          will control the frame rate. -->
+        <updateRate>0.0</updateRate>
+        <cameraName>camera_ir</cameraName>
+        <imageTopicName>/camera/color/image_raw</imageTopicName>
+        <cameraInfoTopicName>/camera/color/camera_info</cameraInfoTopicName>
+        <depthImageTopicName>/camera/depth/image_raw</depthImageTopicName>
+        <depthImageCameraInfoTopicName>/camera/depth/camera_info</depthImageCameraInfoTopicName>
+        <pointCloudTopicName>/camera/depth/points</pointCloudTopicName>
+        <frameName>camera_link</frameName>
+        <pointCloudCutoff>0.5</pointCloudCutoff>
+        <pointCloudCutoffMax>3.0</pointCloudCutoffMax>
+        <distortionK1>0</distortionK1>
+        <distortionK2>0</distortionK2>
+        <distortionK3>0</distortionK3>
+        <distortionT1>0</distortionT1>
+        <distortionT2>0</distortionT2>
+        <CxPrime>0</CxPrime>
+        <Cx>0</Cx>
+        <Cy>0</Cy>
+        <focalLength>0</focalLength>
+        <hackBaseline>0</hackBaseline>
+      </plugin>
+    </sensor>
+  </gazebo>
+  <joint name="camera_joint" type="fixed">
+    <parent link="tool0" />
+    <child link = "camera_link" />
+    <origin xyz="0.0 0.0 0.0" rpy="0.0 ${-pi/2} ${pi/2}" />
+  </joint>
   <link name="world" />
   <joint name="world_joint" type="fixed">

Commit message: working alpha v2.0

File: urdf/golf_club.urdf.xacro (robot description, xacro)
@@ -36,5 +36,5 @@
         <kp>500000</kp>
         <kd>0</kd>
-        <minDepth>0</minDepth>
+        <minDepth>0.001</minDepth>
         <maxVel>1000</maxVel>
     </gazebo>

File: urdf/ur5.urdf.xacro (robot description, xacro)
@@ -101,11 +101,11 @@
       <axis xyz="0 0 1" />
       <xacro:unless value="${joint_limited}">
-        <limit lower="${-2.0 * pi}" upper="${2.0 * pi}" effort="300.0" velocity="6.28"/>
-        <xacro:if value="${safety_limits}">
-          <safety_controller soft_lower_limit="${-2.0 * pi + safety_pos_margin}" soft_upper_limit="${2.0 * pi - safety_pos_margin}" k_position="${safety_k_position}" k_velocity="0.0"/>
-        </xacro:if>
-      </xacro:unless>
-      <xacro:if value="${joint_limited}">
-        <limit lower="${shoulder_pan_lower_limit}" upper="${shoulder_pan_upper_limit}" effort="300.0" velocity="6.28"/>
+        <limit lower="${-2.0 * pi}" upper="${2.0 * pi}" effort="500.0" velocity="9.42"/>
+        <xacro:if value="${safety_limits}">
+          <safety_controller soft_lower_limit="${-2.0 * pi + safety_pos_margin}" soft_upper_limit="${2.0 * pi - safety_pos_margin}" k_position="${safety_k_position}" k_velocity="0.0"/>
+        </xacro:if>
+      </xacro:unless>
+      <xacro:if value="${joint_limited}">
+        <limit lower="${shoulder_pan_lower_limit}" upper="${shoulder_pan_upper_limit}" effort="500.0" velocity="9.42"/>
         <xacro:if value="${safety_limits}">
           <safety_controller soft_lower_limit="${shoulder_pan_lower_limit + safety_pos_margin}" soft_upper_limit="${shoulder_pan_upper_limit - safety_pos_margin}" k_position="${safety_k_position}" k_velocity="0.0"/>

Commit message: biggest update, more realistic swing

File: urdf/golf_club.urdf.xacro (robot description, xacro)
@@ -9,5 +9,5 @@
         <link name="${prefix}_golf_club">
             <visual>
-                <origin rpy="${pi} ${pi/2} 0" xyz="0.0 0.6 0.0" />
+                <origin rpy="${-pi/2} 0 ${pi}" xyz="0.0 0.0 0.6" />
                 <geometry>
                     <mesh scale="0.005 0.005 0.005" filename="package://golfbot/meshes/golf_club.stl"/>
@@ -15,5 +15,5 @@
             </visual>
             <collision>
-                <origin rpy="${pi} ${pi/2} 0" xyz="0.0 0.6 0.0" />
+                <origin rpy="${-pi/2} 0 ${pi}" xyz="0.0 0.0 0.6" />
                 <geometry>
                     <mesh scale="0.005 0.005 0.005" filename="package://golfbot/meshes/golf_club.stl"/>

File: urdf/ur5_robot.urdf.xacro (robot description, xacro)
@@ -7,5 +7,4 @@
   <!-- ur5 -->
   <xacro:include filename="$(find golfbot)/urdf/ur5.urdf.xacro" />
-  <xacro:include filename="golf_club.urdf.xacro" />
   <!-- arm -->
   <xacro:ur5_robot prefix="" joint_limited="false"
@@ -13,5 +12,8 @@
   />
   <!-- golf club -->
-  <xacro:golf_club prefix="" connected_to="tool0" />
+  <xacro:include filename="golf_club.urdf.xacro" />
+  <!-- <xacro:golf_club prefix="" connected_to="tool0" /> -->
+  <!-- ddrive -->
+  <xacro:include filename="ddrive.urdf.xacro" />
   <!-- camera link -->
   <xacro:include filename="$(find golfbot)/urdf/_d435.urdf.xacro" />
@@ -25,3 +27,8 @@
     <origin xyz="0.0 0.0 0.0" rpy="0.0 0.0 0.0" />
   </joint>
+  <joint name="ddrive_joint" type="fixed">
+    <parent link="base_link" />
+    <child link = "ddrive_base_link" />
+    <origin xyz="0.0 0.0 5.0" rpy="0.0 0.0 0.0" />
+  </joint>
 </robot>

Commit message: analytical solution

File: urdf/golf_club.urdf.xacro (robot description, xacro)
@@ -27,6 +27,6 @@
             </collision>
             <inertial>
-                <mass value="10"/>
-                <inertia ixx="10.0" ixy="0.0" ixz="0.0" iyy="0.0" iyz="0.0" izz="10.0"/>
+                <mass value="0.5"/>
+                <inertia ixx="1.0" ixy="0.0" ixz="0.0" iyy="0.0" iyz="0.0" izz="1.0"/>
             </inertial>
         </link>

File: urdf/golfbot.urdf.xacro (robot description, xacro)
@@ -18,5 +18,5 @@
     <parent link="ddrive_base_link" />
     <child link = "base_link" />
-    <origin xyz="0.0 0.2 0.4" rpy="0.0 0.0 ${pi/2}" />
+    <origin xyz="0.0 0.2 0.35" rpy="0.0 0.0 ${pi/2}" />
   </joint>
   <!-- weight block-->
@@ -45,7 +45,7 @@
     <link name="arm_support">
         <visual>
-            <origin rpy="0 0.0 0.0" xyz="0 0.2 0.2" />
+            <origin rpy="0 0.0 0.0" xyz="0 0.2 0.175" />
             <geometry>
-                <cylinder radius="0.05" length="0.4"/>
+                <cylinder radius="0.05" length="0.35"/>
             </geometry>
             <material name="green"/>
@@ -67,7 +67,7 @@
     <link name="camera_support">
         <visual>
-            <origin rpy="0 0.0 0.0" xyz="0 0 0.35" />
+            <origin rpy="0 0.0 0.0" xyz="0 0 0.4" />
             <geometry>
-                <cylinder radius="0.01" length="0.7"/>
+                <cylinder radius="0.01" length="0.8"/>
             </geometry>
             <material name="green"/>
@@ -89,5 +89,5 @@
   <xacro:include filename="$(find golfbot)/urdf/_d435.urdf.xacro" />
   <xacro:sensor_d435 name="camera" topics_ns="camera" parent="camera_support" publish_pointcloud="true">
-    <origin xyz="0 0 0.7" rpy="0 0 ${pi}" />
+    <origin xyz="0 0 0.8" rpy="0 0 ${pi}" />
   </xacro:sensor_d435>
 </robot>
